File: FK_fpga_shield/_autosave-FK_fpga_shield.kicad_pcb (KiCad board)
At the start: 2 copper layers, 136 parts, among them J0 USB_B_Mini, J1 molex-51382-0400-microclasp, J10 molex-51382-0400-microclasp, J11 molex-51382-0400-microclasp, J12 molex-51382-0400-microclasp, J13 molex-51382-0400-microclasp, J14 molex-51382-0400-microclasp, J15 molex-51382-0400-microclasp, J16 molex-51382-0400-microclasp, J17 molex-51382-0400-microclasp, J18 molex-51382-0400-microclasp, J19 molex-51382-0400-microclasp, J2 molex-51382-0400-microclasp, J20 molex-51382-0400-microclasp, J21 molex-51382-0400-microclasp, J22 molex-51382-0400-microclasp, J23 molex-51382-0400-microclasp, J24 molex-51382-0400-microclasp, J25 molex-51382-0400-microclasp, J26 molex-51382-0400-microclasp, J27 molex-51382-0400-microclasp, J28 molex-51382-0400-microclasp, J29 molex-51382-0400-microclasp, J3 molex-51382-0400-microclasp, J30 molex-51382-0400-microclasp, J31 molex-51382-0400-microclasp, J32 molex-51382-0400-microclasp, J33 molex-51382-0400-microclasp, J34 molex-51382-0400-microclasp, J35 molex-51382-0400-microclasp, J4 molex-51382-0400-microclasp, J5 molex-51382-0400-microclasp, J6 molex-51382-0400-microclasp, J7 molex-51382-0400-microclasp, J8 molex-51382-0400-microclasp, J9 molex-51382-0400-microclasp, U1 FT232RL, U2 nvt2010pw, U3 nvt2010pw, U4 nvt2010pw, U5 nvt2010pw, U6 nvt2010pw, U7 nvt2010pw, U8 nvt2010pw

Commit message: WIP fpga shield layout
Parts:
- moved C6 349.4 mm to (345.1, 24.9)
- moved R44 349.4 mm to (345.1, 27.8)
- moved R79 349.4 mm to (349.9, 33.7)
- moved C2 349.4 mm to (360.3, 55.8)
- moved C4 349.4 mm to (365.1, 55.8)
- moved C7 349.4 mm to (334.1, 35.7)
- moved C8 349.4 mm to (329.4, 38.6)
- moved J0 349.4 mm to (277.9, 43.8)
- moved R1 349.4 mm to (360.3, 58.7)
- moved R17 349.4 mm to (329.4, 35.7)
- moved R2 349.4 mm to (365.1, 58.7)
- moved R26 349.4 mm to (343.6, 42.5)
- moved R49 349.4 mm to (338.9, 35.7)
- moved R54 349.4 mm to (348.4, 36.6)
- moved R58 349.4 mm to (338.9, 41.6)
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- renumbered J15 to J11, J14 to J12, J12 to J14, J11 to J15, J20 to J16, J19 to J17, J17 to J19, J16 to J20
Routing:
- net Net-(J10-Pad2): track 0.00 -> 34.1 mm
