File: FK_fpga_shield/FK_fpga_shield.sch (KiCad schematic (older format))
At the start: 157 parts, among them J0 USB_B_Mini, J1 molex-51382-0400-microclasp, J10 molex-51382-0400-microclasp, J11 molex-51382-0400-microclasp, J12 molex-51382-0400-microclasp, J13 molex-51382-0400-microclasp, J14 molex-51382-0400-microclasp, J15 molex-51382-0400-microclasp, J16 molex-51382-0400-microclasp, J17 molex-51382-0400-microclasp, J18 molex-51382-0400-microclasp, J19 molex-51382-0400-microclasp, J2 molex-51382-0400-microclasp, J20 molex-51382-0400-microclasp, J21 molex-51382-0400-microclasp, J22 molex-51382-0400-microclasp, J23 molex-51382-0400-microclasp, J24 molex-51382-0400-microclasp, J25 molex-51382-0400-microclasp, J26 molex-51382-0400-microclasp, J27 molex-51382-0400-microclasp, J28 molex-51382-0400-microclasp, J29 molex-51382-0400-microclasp, J3 molex-51382-0400-microclasp, J30 molex-51382-0400-microclasp, J31 molex-51382-0400-microclasp, J32 molex-51382-0400-microclasp, J33 molex-51382-0400-microclasp, J34 molex-51382-0400-microclasp, J35 molex-51382-0400-microclasp, J36 Barrel_Jack_MountingPin, J4 molex-51382-0400-microclasp, J5 molex-51382-0400-microclasp, J6 molex-51382-0400-microclasp, J7 molex-51382-0400-microclasp, J8 molex-51382-0400-microclasp, J9 molex-51382-0400-microclasp, U1 FT232RL, U2 nvt2010pw, U3 nvt2010pw, U4 nvt2010pw, U5 nvt2010pw, U6 nvt2010pw, U7 nvt2010pw, U8 nvt2010pw, Y1 DNP_(12MHz)

Commit message: choosen choke
Parts:
- added C31: DNP_1n, Capacitor_SMD:C_0805_2012Metric_Pad1.15x1.40mm_HandSolder, symbol Device:C_Small
- added H3, H4, H5, H6: MountingHole, MountingHole:MountingHole_3mm, symbol Mechanical:MountingHole
- added L1: WE_744823422, Inductor_THT:L_CommonMode_Wuerth_WE-CMB-M, symbol Device:L_Core_Iron_Coupled_1243
- gave numbers to parts that had none: 5
Connections:
- net 5V: now also C31.2, L1.3; no longer J36.1
- net GND: now also C31.1, L1.2; no longer J36.2, J36.MP (MountPin)
- new net: J36.1, L1.4
- new net: J36.2, J36.MP (MountPin), L1.1
Other:
- moved on the sheet: J36
Changed lines of the file:
@@
 L power:GND #PWR0112
 U 1 1 61D45B36
-P 9400 7000
-F 0 "#PWR0112" H 9400 6750 50  0001 C CNN
-F 1 "GND" H 9405 6827 50  0000 C CNN
-F 2 "" H 9400 7000 50  0001 C CNN
-F 3 "" H 9400 7000 50  0001 C CNN
-	1    9400 7000
+P 9600 7000
+F 0 "#PWR0112" H 9600 6750 50  0001 C CNN
+F 1 "GND" H 9605 6827 50  0000 C CNN
+F 2 "" H 9600 7000 50  0001 C CNN
+F 3 "" H 9600 7000 50  0001 C CNN
+	1    9600 7000
 	1    0    0    -1
 $EndComp
 Text Label 9600 6300 0    50   ~ 0
 5V
-Wire Wire Line
-	9500 6500 9600 6500
 Text Label 12950 6950 3    50   ~ 0
 35a
@@
 	9600 6500 9600 6300
 Wire Wire Line
-	9500 6700 9600 6700
-Wire Wire Line
 	9600 6500 9850 6500
 Connection ~ 9600 6500
@@
 L Connector:Barrel_Jack_MountingPin J36
 U 1 1 60468A7D
-P 9200 6600
-F 0 "J36" H 9257 6917 50  0000 C CNN
-F 1 "Barrel_Jack_MountingPin" H 9257 6826 50  0000 C CNN
-F 2 "Connector_BarrelJack:BarrelJack_CUI_PJ-063AH_Horizontal" H 9250 6560 50  0001 C CNN
-F 3 "~" H 9250 6560 50  0001 C CNN
-	1    9200 6600
-	1    0    0    -1
-$EndComp
-Wire Wire Line
-	9200 6900 9400 6900
-Wire Wire Line
-	9400 6900 9400 7000
-Wire Wire Line
-	9400 6900 9600 6900
-Wire Wire Line
-	9600 6700 9600 6900
-Connection ~ 9400 6900
+P 7750 6600
+F 0 "J36" H 7807 6917 50  0000 C CNN
+F 1 "Barrel_Jack_MountingPin" H 7807 6826 50  0000 C CNN
+F 2 "Connector_BarrelJack:BarrelJack_CUI_PJ-063AH_Horizontal" H 7800 6560 50  0001 C CNN
+F 3 "~" H 7800 6560 50  0001 C CNN
+	1    7750 6600
+	1    0    0    -1
+$EndComp
 $Comp
 L Device:C_Small C20
@@
 Connection ~ 10550 6700
 $Comp
-L Device:C_Small C?
+L Device:C_Small C26
 U 1 1 607ED0DA
 P 10750 6600
-F 0 "C?" H 10700 6400 50  0000 L CNN
+F 0 "C26" H 10700 6400 50  0000 L CNN
 F 1 "1u_MCC" H 10650 6300 50  0000 L CNN
 F 2 "Capacitor_SMD:C_0805_2012Metric_Pad1.15x1.40mm_HandSolder" H 10750 6600 50  0001 C CNN
@@
 Connection ~ 10750 6700
 $Comp
-L Device:C_Small C?
+L Device:C_Small C27
 U 1 1 609644C2
 P 11000 6600
-F 0 "C?" H 10950 6400 50  0000 L CNN
+F 0 "C27" H 10950 6400 50  0000 L CNN
 F 1 "DNP_10n" V 11000 6000 50  0000 L CNN
 F 2 "Capacitor_SMD:C_0805_2012Metric_Pad1.15x1.40mm_HandSolder" H 11000 6600 50  0001 C CNN
@@
 	11000 6500 11150 6500
 $Comp
-L Device:C_Small C?
+L Device:C_Small C28
 U 1 1 609CA4EF
 P 11150 6600
-F 0 "C?" H 11100 6400 50  0000 L CNN
+F 0 "C28" H 11100 6400 50  0000 L CNN
 F 1 "DNP_10n" V 11150 6000 50  0000 L CNN
 F 2 "Capacitor_SMD:C_0805_2012Metric_Pad1.15x1.40mm_HandSolder" H 11150 6600 50  0001 C CNN
@@
 	11150 6500 11300 6500
 $Comp
-L Device:C_Small C?
+L Device:C_Small C29
 U 1 1 609CA843
 P 11300 6600
-F 0 "C?" H 11250 6400 50  0000 L CNN
+F 0 "C29" H 11250 6400 50  0000 L CNN
 F 1 "DNP_1n" V 11300 6000 50  0000 L CNN
 F 2 "Capacitor_SMD:C_0805_2012Metric_Pad1.15x1.40mm_HandSolder" H 11300 6600 50  0001 C CNN
@@
 	11300 6500 11450 6500
 $Comp
-L Device:C_Small C?
+L Device:C_Small C30
 U 1 1 609CAA01
 P 11450 6600
-F 0 "C?" H 11400 6400 50  0000 L CNN
+F 0 "C30" H 11400 6400 50  0000 L CNN
 F 1 "DNP_1n" V 11450 6000 50  0000 L CNN
 F 2 "Capacitor_SMD:C_0805_2012Metric_Pad1.15x1.40mm_HandSolder" H 11450 6600 50  0001 C CNN
@@
 $EndComp
 Connection ~ 11450 6700
-Wire Wire Line
-	11450 6700 11550 6700
 Connection ~ 11450 6500
-Wire Wire Line
-	11450 6500 11550 6500
+$Comp
+L Device:C_Small C31
+U 1 1 604B11B4
+P 11600 6600
+F 0 "C31" H 11550 6400 50  0000 L CNN
+F 1 "DNP_1n" V 11600 6000 50  0000 L CNN
+F 2 "Capacitor_SMD:C_0805_2012Metric_Pad1.15x1.40mm_HandSolder" H 11600 6600 50  0001 C CNN
+F 3 "~" H 11600 6600 50  0001 C CNN
+	1    11600 6600
+	-1   0    0    1
+$EndComp
+Wire Wire Line
+	11450 6500 11600 6500
+Wire Wire Line
+	11450 6700 11600 6700
+$Comp
+L Mechanical:MountingHole H3
+U 1 1 606CC2D0
+P 10100 5050
+F 0 "H3" H 10200 5096 50  0000 L CNN
+F 1 "MountingHole" H 10200 5005 50  0000 L CNN
+F 2 "MountingHole:MountingHole_3mm" H 10100 5050 50  0001 C CNN
+F 3 "~" H 10100 5050 50  0001 C CNN
+	1    10100 5050
+	1    0    0    -1
+$EndComp
+$Comp
+L Mechanical:MountingHole H4
+U 1 1 606CCE4C
+P 10100 5250
+F 0 "H4" H 10200 5296 50  0000 L CNN
+F 1 "MountingHole" H 10200 5205 50  0000 L CNN
+F 2 "MountingHole:MountingHole_3mm" H 10100 5250 50  0001 C CNN
+F 3 "~" H 10100 5250 50  0001 C CNN
+	1    10100 5250
+	1    0    0    -1
+$EndComp
+$Comp
+L Mechanical:MountingHole H6
+U 1 1 6078AF04
+P 10100 5650
+F 0 "H6" H 10200 5696 50  0000 L CNN
+F 1 "MountingHole" H 10200 5605 50  0000 L CNN
+F 2 "MountingHole:MountingHole_3mm" H 10100 5650 50  0001 C CNN
+F 3 "~" H 10100 5650 50  0001 C CNN
+	1    10100 5650
+	1    0    0    -1
+$EndComp
+$Comp
+L Mechanical:MountingHole H5
+U 1 1 6072BEC8
+P 10100 5450
+F 0 "H5" H 10200 5496 50  0000 L CNN
+F 1 "MountingHole" H 10200 5405 50  0000 L CNN
+F 2 "MountingHole:MountingHole_3mm" H 10100 5450 50  0001 C CNN
+F 3 "~" H 10100 5450 50  0001 C CNN
+	1    10100 5450
+	1    0    0    -1
+$EndComp
+$Comp
+L Device:L_Core_Iron_Coupled_1243 L1
+U 1 1 60A35E84
+P 9050 6600
+F 0 "L1" H 9050 6881 50  0000 C CNN
+F 1 "WE_744823422" H 9050 6790 50  0000 C CNN
+F 2 "Inductor_THT:L_CommonMode_Wuerth_WE-CMB-M" H 9050 6600 50  0001 C CNN
+F 3 "~" H 9050 6600 50  0001 C CNN
+	1    9050 6600
+	1    0    0    1
+$EndComp
+Wire Wire Line
+	9250 6500 9600 6500
+Wire Wire Line
+	9250 6700 9600 6700
+Wire Wire Line
+	9600 6700 9600 7000
+Wire Wire Line
+	8050 6500 8850 6500
+Wire Wire Line
+	8050 6700 8100 6700
+Wire Wire Line
+	8100 6700 8100 6900
+Wire Wire Line
+	8100 6900 7750 6900
+Connection ~ 8100 6700
+Wire Wire Line
+	8100 6700 8850 6700
 $EndSCHEMATC

Commit message: 2x4 breakout header for uart convertor, choke laid out
Parts:
- added D_RX1: LED RX, LED_SMD:LED_0805_2012Metric_Pad1.15x1.40mm_HandSolder, symbol Device:LED_Small
- added D_TX1: LED_TX, LED_SMD:LED_0805_2012Metric_Pad1.15x1.40mm_HandSolder, symbol Device:LED_Small
- added J37: Conn_02x04_Top_Bottom, Connector_PinHeader_2.54mm:PinHeader_2x04_P2.54mm_Vertical, symbol Connector_Generic:Conn_02x04_Top_Bottom
- added R80, R81: 270, Resistor_SMD:R_0805_2012Metric_Pad1.15x1.40mm_HandSolder, symbol Device:R_Small
Connections:
- net 3V3: now also J37.7 (Pin_7)
- net 5V: now also J37.5 (Pin_5), R80.1, R81.1
- net GND: now also J37.8 (Pin_8)
- net at U1.12 (CBUS4): now also J37.6 (Pin_6)
- net at U1.13 (CBUS2): now also J37.4 (Pin_4)
- net at U1.14 (CBUS3): now also J37.3 (Pin_3)
- net at U1.22 (CBUS1): now also D_RX1.1 (K), J37.2 (Pin_2)
- net at U1.23 (CBUS0): now also D_TX1.1 (K), J37.1 (Pin_1)
- new net: D_TX1.2 (A), R80.2
- new net: D_RX1.2 (A), R81.2
Other:
- note added: "TODO:\nresistor values\nmove choke?\nsilkscreen etc"
- note removed: "todo led indicators"
Changed lines of the file:
@@
 	1    0    0    -1
 $EndComp
-Text Notes 12950 2200 0    50   ~ 0
-todo led indicators
 $Comp
 L FK_fpga_shield_custom_symbols:nvt2010pw U2
@@
 Wire Wire Line
 	8100 6700 8850 6700
+$Comp
+L Device:R_Small R80
+U 1 1 610D1E94
+P 13200 1800
+F 0 "R80" H 13259 1846 50  0000 L CNN
+F 1 "270" H 13259 1755 50  0000 L CNN
+F 2 "Resistor_SMD:R_0805_2012Metric_Pad1.15x1.40mm_HandSolder" H 13200 1800 50  0001 C CNN
+F 3 "~" H 13200 1800 50  0001 C CNN
+	1    13200 1800
+	1    0    0    -1
+$EndComp
+$Comp
+L Device:R_Small R81
+U 1 1 610D21C6
+P 13500 1800
+F 0 "R81" H 13559 1846 50  0000 L CNN
+F 1 "270" H 13559 1755 50  0000 L CNN
+F 2 "Resistor_SMD:R_0805_2012Metric_Pad1.15x1.40mm_HandSolder" H 13500 1800 50  0001 C CNN
+F 3 "~" H 13500 1800 50  0001 C CNN
+	1    13500 1800
+	1    0    0    -1
+$EndComp
+$Comp
+L Device:LED_Small D_TX1
+U 1 1 610D2603
+P 13200 2000
+F 0 "D_TX1" V 13246 1930 50  0000 R CNN
+F 1 "LED_TX" H 13300 2100 50  0000 R CNN
+F 2 "LED_SMD:LED_0805_2012Metric_Pad1.15x1.40mm_HandSolder" V 13200 2000 50  0001 C CNN
+F 3 "~" V 13200 2000 50  0001 C CNN
+	1    13200 2000
+	0    -1   -1   0
+$EndComp
+$Comp
+L Device:LED_Small D_RX1
+U 1 1 610D420B
+P 13500 2000
+F 0 "D_RX1" V 13500 1850 50  0000 R CNN
+F 1 "LED RX" H 13550 1900 50  0000 R CNN
+F 2 "LED_SMD:LED_0805_2012Metric_Pad1.15x1.40mm_HandSolder" V 13500 2000 50  0001 C CNN
+F 3 "~" V 13500 2000 50  0001 C CNN
+	1    13500 2000
+	0    -1   -1   0
+$EndComp
+Wire Wire Line
+	13200 1700 13350 1700
+Wire Wire Line
+	13350 1700 13350 1500
+Wire Wire Line
+	13350 1500 13500 1500
+Connection ~ 13350 1700
+Wire Wire Line
+	13350 1700 13500 1700
+Text Label 13500 1500 0    50   ~ 0
+5V
+Wire Wire Line
+	13200 2100 13200 2400
+Wire Wire Line
+	13200 2400 12750 2400
+Wire Wire Line
+	12750 2500 13500 2500
+Wire Wire Line
+	13500 2500 13500 2100
+$Comp
+L Connector_Generic:Conn_02x04_Top_Bottom J37
+U 1 1 617C9849
+P 13950 2850
+F 0 "J37" H 14000 3167 50  0000 C CNN
+F 1 "Conn_02x04_Top_Bottom" H 14000 3076 50  0000 C CNN
+F 2 "Connector_PinHeader_2.54mm:PinHeader_2x04_P2.54mm_Vertical" H 13950 2850 50  0001 C CNN
+F 3 "~" H 13950 2850 50  0001 C CNN
+	1    13950 2850
+	1    0    0    -1
+$EndComp
+Wire Wire Line
+	13500 2500 13500 2850
+Wire Wire Line
+	13500 2850 13750 2850
+Connection ~ 13500 2500
+Wire Wire Line
+	13200 2400 13650 2400
+Wire Wire Line
+	13650 2400 13650 2750
+Wire Wire Line
+	13650 2750 13750 2750
+Connection ~ 13200 2400
+Wire Wire Line
+	13750 2950 13200 2950
+Wire Wire Line
+	13200 2950 13200 2700
+Wire Wire Line
+	13200 2700 12750 2700
+Wire Wire Line
+	13750 3050 13350 3050
+Wire Wire Line
+	13350 3050 13350 2600
+Wire Wire Line
+	13350 2600 12750 2600
+Wire Wire Line
+	14250 2850 14400 2850
+Wire Wire Line
+	14400 2850 14400 3200
+Wire Wire Line
+	14400 3200 12750 3200
+Wire Wire Line
+	12750 3200 12750 2800
+Text Label 14250 2750 0    50   ~ 0
+5V
+$Comp
+L power:GND #PWR0114
+U 1 1 61AAB2C6
+P 14250 3050
+F 0 "#PWR0114" H 14250 2800 50  0001 C CNN
+F 1 "GND" H 14250 2850 50  0000 C CNN
+F 2 "" H 14250 3050 50  0001 C CNN
+F 3 "" H 14250 3050 50  0001 C CNN
+	1    14250 3050
+	1    0    0    -1
+$EndComp
+Text Label 14250 2950 0    50   ~ 0
+3V3
+Text Notes 4600 8300 0    1181 ~ 0
+TODO:\nresistor values\nmove choke?\nsilkscreen etc
 $EndSCHEMATC

Commit message: replace common mode choke with filter
Parts:
- removed C1, C10, C11, C14, C15, C16, C17, C18, C19, C2, C20, C25, C3, C5, C6, C7, C8, C9: 100n, Capacitor_SMD:C_0805_2012Metric_Pad1.15x1.40mm_HandSolder, symbol Device:C_Small
- removed C12, C13: dnp, Capacitor_SMD:C_0805_2012Metric_Pad1.15x1.40mm_HandSolder, symbol Device:C_Small
- removed C21, C22, C23, C24: 22u, Capacitor_THT:CP_Radial_D6.3mm_P2.50mm, symbol Device:CP_Small
- removed C26: 1u_MCC, Capacitor_SMD:C_0805_2012Metric_Pad1.15x1.40mm_HandSolder, symbol Device:C_Small
- removed C27, C28: DNP_10n, Capacitor_SMD:C_0805_2012Metric_Pad1.15x1.40mm_HandSolder, symbol Device:C_Small
- removed C29, C30, C31: DNP_1n, Capacitor_SMD:C_0805_2012Metric_Pad1.15x1.40mm_HandSolder, symbol Device:C_Small
- removed C4: 4.7u, Capacitor_SMD:C_0805_2012Metric_Pad1.15x1.40mm_HandSolder, symbol Device:CP_Small
- removed D_RX1: LED RX, LED_SMD:LED_0805_2012Metric_Pad1.15x1.40mm_HandSolder, symbol Device:LED_Small
- removed D_TX1: LED_TX, LED_SMD:LED_0805_2012Metric_Pad1.15x1.40mm_HandSolder, symbol Device:LED_Small
- removed H1, H2: Conn_02x20_Odd_Even, Connector_PinSocket_2.54mm:PinSocket_2x20_P2.54mm_Vertical, symbol Connector_Generic:Conn_02x20_Odd_Even
- removed H3, H4, H5, H6: MountingHole, MountingHole:MountingHole_3mm, symbol Mechanical:MountingHole
- removed J0: USB_B_Mini, 54819-0519:54819-0519, symbol Connector:USB_B_Mini
- removed J1, J10, J11, J12, J13, J14, J15, J16, J17, J18, J19, J2, J20, J21, J22, J23, J24, J25, J26, J27, J28, J29, J3, J30, J31, J32, J33, J34, J35, J4, J5, J6, J7, J8, J9: molex-51382-0400-microclasp, FK_fpga_shield_custom_footprints:Molex_MicroClasp_55935-0410_1x04_P2.00mm_Horizontal_3DMODEL, symbol FK_fpga_shield_custom_symbols:molex-51382-0400-microclasp
- removed J36: Barrel_Jack_MountingPin, Connector_BarrelJack:BarrelJack_CUI_PJ-063AH_Horizontal, symbol Connector:Barrel_Jack_MountingPin
- removed J37: Conn_02x04_Top_Bottom, Connector_PinHeader_2.54mm:PinHeader_2x04_P2.54mm_Vertical, symbol Connector_Generic:Conn_02x04_Top_Bottom
- removed L1: WE_744823422, Inductor_THT:L_CommonMode_Wuerth_WE-CMB-M, symbol Device:L_Core_Iron_Coupled_1243
- removed R1: 4k7, Resistor_SMD:R_0805_2012Metric_Pad1.15x1.40mm_HandSolder, symbol Device:R_Small
- removed R10, R11, R12, R13, R14, R15, R16, R17, R18, R19, R20, R21, R22, R23, R24, R25, R26, R27, R28, R29, R3, R30, R31, R32, R33, R34, R35, R36, R37, R38, R39, R4, R40, R41, R42, R43, R44, R45, R46, R47, R48, R49, R5, R50, R51, R52, R58, R59, R6, R60, R61, R62, R63, R64, R65, R66, R67, R68, R69, R7, R70, R71, R72, R73, R74, R75, R76, R77, R8, R9: 5k6, Resistor_SMD:R_0805_2012Metric_Pad1.15x1.40mm_HandSolder, symbol Device:R_Small
- removed R2: 10k, Resistor_SMD:R_0805_2012Metric_Pad1.15x1.40mm_HandSolder, symbol Device:R_Small
- removed R53, R54, R55, R56, R57, R78, R79: 200k, Resistor_SMD:R_0805_2012Metric_Pad1.15x1.40mm_HandSolder, symbol Device:R_Small
- removed R80, R81: 270, Resistor_SMD:R_0805_2012Metric_Pad1.15x1.40mm_HandSolder, symbol Device:R_Small
- removed U1: FT232RL, Package_SO:SSOP-28_5.3x10.2mm_P0.65mm, symbol Interface_USB:FT232RL
- removed U2, U3, U4, U5, U6, U7, U8: nvt2010pw, Package_SO:TSSOP-24_4.4x7.8mm_P0.65mm, symbol FK_fpga_shield_custom_symbols:nvt2010pw
- removed Y1: DNP_(12MHz), Crystal:Crystal_SMD_HC49-SD, symbol Device:Crystal
Other:
- note removed: "External oscillator not reqired\nper datasheet when 5V powered.\nFootprint added anyway just in case."
- note removed: "TODO:\nresistor values\nmove choke?\nsilkscreen etc"

Commit message: restore schematic from last version
Parts:
- added C1, C10, C11, C14, C15, C16, C17, C18, C19, C2, C20, C25, C3, C5, C6, C7, C8, C9: 100n, Capacitor_SMD:C_0805_2012Metric_Pad1.15x1.40mm_HandSolder, symbol Device:C_Small
- added C12, C13: dnp, Capacitor_SMD:C_0805_2012Metric_Pad1.15x1.40mm_HandSolder, symbol Device:C_Small
- added C21, C22, C23, C24: 22u, Capacitor_THT:CP_Radial_D6.3mm_P2.50mm, symbol Device:CP_Small
- added C26: 1u_MCC, Capacitor_SMD:C_0805_2012Metric_Pad1.15x1.40mm_HandSolder, symbol Device:C_Small
- added C27, C28: DNP_10n, Capacitor_SMD:C_0805_2012Metric_Pad1.15x1.40mm_HandSolder, symbol Device:C_Small
- added C29, C30, C31: DNP_1n, Capacitor_SMD:C_0805_2012Metric_Pad1.15x1.40mm_HandSolder, symbol Device:C_Small
- added C4: 4.7u, Capacitor_SMD:C_0805_2012Metric_Pad1.15x1.40mm_HandSolder, symbol Device:CP_Small
- added D_RX1: LED RX, LED_SMD:LED_0805_2012Metric_Pad1.15x1.40mm_HandSolder, symbol Device:LED_Small
- added D_TX1: LED_TX, LED_SMD:LED_0805_2012Metric_Pad1.15x1.40mm_HandSolder, symbol Device:LED_Small
- added H1, H2: Conn_02x20_Odd_Even, Connector_PinSocket_2.54mm:PinSocket_2x20_P2.54mm_Vertical, symbol Connector_Generic:Conn_02x20_Odd_Even
- added H3, H4, H5, H6: MountingHole, MountingHole:MountingHole_3mm, symbol Mechanical:MountingHole
- added J0: USB_B_Mini, 54819-0519:54819-0519, symbol Connector:USB_B_Mini
- added J1, J10, J11, J12, J13, J14, J15, J16, J17, J18, J19, J2, J20, J21, J22, J23, J24, J25, J26, J27, J28, J29, J3, J30, J31, J32, J33, J34, J35, J4, J5, J6, J7, J8, J9: molex-51382-0400-microclasp, FK_fpga_shield_custom_footprints:Molex_MicroClasp_55935-0410_1x04_P2.00mm_Horizontal_3DMODEL, symbol FK_fpga_shield_custom_symbols:molex-51382-0400-microclasp
- added J36: Barrel_Jack_MountingPin, Connector_BarrelJack:BarrelJack_CUI_PJ-063AH_Horizontal, symbol Connector:Barrel_Jack_MountingPin
- added J37: Conn_02x04_Top_Bottom, Connector_PinHeader_2.54mm:PinHeader_2x04_P2.54mm_Vertical, symbol Connector_Generic:Conn_02x04_Top_Bottom
- added L1: WE_744823422, Inductor_THT:L_CommonMode_Wuerth_WE-CMB-M, symbol Device:L_Core_Iron_Coupled_1243
- added R1: 4k7, Resistor_SMD:R_0805_2012Metric_Pad1.15x1.40mm_HandSolder, symbol Device:R_Small
- added R10, R11, R12, R13, R14, R15, R16, R17, R18, R19, R20, R21, R22, R23, R24, R25, R26, R27, R28, R29, R3, R30, R31, R32, R33, R34, R35, R36, R37, R38, R39, R4, R40, R41, R42, R43, R44, R45, R46, R47, R48, R49, R5, R50, R51, R52, R58, R59, R6, R60, R61, R62, R63, R64, R65, R66, R67, R68, R69, R7, R70, R71, R72, R73, R74, R75, R76, R77, R8, R9: 5k6, Resistor_SMD:R_0805_2012Metric_Pad1.15x1.40mm_HandSolder, symbol Device:R_Small
- added R2: 10k, Resistor_SMD:R_0805_2012Metric_Pad1.15x1.40mm_HandSolder, symbol Device:R_Small
- added R53, R54, R55, R56, R57, R78, R79: 200k, Resistor_SMD:R_0805_2012Metric_Pad1.15x1.40mm_HandSolder, symbol Device:R_Small
- added R80, R81: 270, Resistor_SMD:R_0805_2012Metric_Pad1.15x1.40mm_HandSolder, symbol Device:R_Small
- added U1: FT232RL, Package_SO:SSOP-28_5.3x10.2mm_P0.65mm, symbol Interface_USB:FT232RL
- added U2, U3, U4, U5, U6, U7, U8: nvt2010pw, Package_SO:TSSOP-24_4.4x7.8mm_P0.65mm, symbol FK_fpga_shield_custom_symbols:nvt2010pw
- added Y1: DNP_(12MHz), Crystal:Crystal_SMD_HC49-SD, symbol Device:Crystal
Connections:
- new net: J5.2 (C_A), R3.2, U2.13 (B10)
- new net: J5.4 (C_B), R8.2, U2.14 (B9)
- new net: J4.2 (C_A), R13.2, U2.15 (B8)
- new net: J4.4 (C_B), R18.2, U2.16 (B7)
- new net: J3.2 (C_A), R23.2, U2.17 (B6)
- new net: J3.4 (C_B), R28.2, U2.18 (B5)
- new net: J2.2 (C_A), R33.2, U2.19 (B4)
- new net: J2.4 (C_B), R38.2, U2.20 (B3)
- new net: J1.2 (C_A), R43.2, U2.21 (B2)
- new net: J1.4 (C_B), R48.2, U2.22 (B1)
- new net: C5.1, R53.2, U2.23 (VrefB), U2.24 (EN)
- new net: J37.6 (Pin_6), U1.12 (CBUS4)
- new net: J37.4 (Pin_4), U1.13 (CBUS2)
- new net: J37.3 (Pin_3), U1.14 (CBUS3)
- new net: J0.3 (D+), U1.15 (USBD+)
- new net: J0.2 (D-), U1.16 (USBD-)
- new net: C1.1, U1.17 (3V3OUT), U1.4 (VCCIO)
- new net: R1.2, R2.1, U1.19 (~RESET~)
- new net: D_RX1.1 (K), J37.2 (Pin_2), U1.22 (CBUS1)
- new net: D_TX1.1 (K), J37.1 (Pin_1), U1.23 (CBUS0)
- new net: C12.1, U1.27 (OSCI), Y1.1
- new net: C13.1, U1.28 (OSCO), Y1.2
- new net: J0.1 (VBUS), R1.1
- new net: J36.1, L1.4
- new net: J36.2, J36.MP (MountPin), L1.1
- new net: J10.2 (C_A), R4.2, U3.13 (B10)
- new net: J10.4 (C_B), R9.2, U3.14 (B9)
- new net: J9.2 (C_A), R14.2, U3.15 (B8)
- new net: J9.4 (C_B), R19.2, U3.16 (B7)
- new net: J8.2 (C_A), R24.2, U3.17 (B6)
- new net: J8.4 (C_B), R29.2, U3.18 (B5)
- new net: J7.2 (C_A), R34.2, U3.19 (B4)
- new net: J7.4 (C_B), R39.2, U3.20 (B3)
- new net: J6.2 (C_A), R44.2, U3.21 (B2)
- new net: J6.4 (C_B), R49.2, U3.22 (B1)
- new net: C6.1, R54.2, U3.23 (VrefB), U3.24 (EN)
- new net: J15.2 (C_A), R5.2, U4.13 (B10)
- new net: J15.4 (C_B), R10.2, U4.14 (B9)
- new net: J14.2 (C_A), R15.2, U4.15 (B8)
- new net: J14.4 (C_B), R20.2, U4.16 (B7)
- new net: J13.2 (C_A), R25.2, U4.17 (B6)
- new net: J13.4 (C_B), R30.2, U4.18 (B5)
- new net: J12.2 (C_A), R35.2, U4.19 (B4)
- new net: J12.4 (C_B), R40.2, U4.20 (B3)
- new net: J11.2 (C_A), R45.2, U4.21 (B2)
- new net: J11.4 (C_B), R50.2, U4.22 (B1)
- new net: C7.1, R55.2, U4.23 (VrefB), U4.24 (EN)
- new net: J20.2 (C_A), R6.2, U5.13 (B10)
- new net: J20.4 (C_B), R11.2, U5.14 (B9)
- new net: J19.2 (C_A), R16.2, U5.15 (B8)
- new net: J19.4 (C_B), R21.2, U5.16 (B7)
- new net: J18.2 (C_A), R26.2, U5.17 (B6)
- new net: J18.4 (C_B), R31.2, U5.18 (B5)
- new net: J17.2 (C_A), R36.2, U5.19 (B4)
- new net: J17.4 (C_B), R41.2, U5.20 (B3)
- new net: J16.2 (C_A), R46.2, U5.21 (B2)
- new net: J16.4 (C_B), R51.2, U5.22 (B1)
- new net: C8.1, R56.2, U5.23 (VrefB), U5.24 (EN)
- new net: J25.2 (C_A), R7.2, U6.13 (B10)
- new net: J25.4 (C_B), R12.2, U6.14 (B9)
- new net: J24.2 (C_A), R17.2, U6.15 (B8)
- new net: J24.4 (C_B), R22.2, U6.16 (B7)
- new net: J23.2 (C_A), R27.2, U6.17 (B6)
- new net: J23.4 (C_B), R32.2, U6.18 (B5)
- new net: J22.2 (C_A), R37.2, U6.19 (B4)
- new net: J22.4 (C_B), R42.2, U6.20 (B3)
- new net: J21.2 (C_A), R47.2, U6.21 (B2)
- new net: J21.4 (C_B), R52.2, U6.22 (B1)
- new net: C9.1, R57.2, U6.23 (VrefB), U6.24 (EN)
- new net: J30.2 (C_A), R58.2, U7.13 (B10)
- new net: J30.4 (C_B), R60.2, U7.14 (B9)
- new net: J29.2 (C_A), R62.2, U7.15 (B8)
- new net: J29.4 (C_B), R64.2, U7.16 (B7)
- new net: J28.2 (C_A), R66.2, U7.17 (B6)
- new net: J28.4 (C_B), R68.2, U7.18 (B5)
- new net: J27.2 (C_A), R70.2, U7.19 (B4)
- new net: J27.4 (C_B), R72.2, U7.20 (B3)
- new net: J26.2 (C_A), R74.2, U7.21 (B2)
- new net: J26.4 (C_B), R76.2, U7.22 (B1)
- new net: C10.1, R78.2, U7.23 (VrefB), U7.24 (EN)
- new net: J35.2 (C_A), R59.2, U8.13 (B10)
- new net: J35.4 (C_B), R61.2, U8.14 (B9)
- new net: J34.2 (C_A), R63.2, U8.15 (B8)
- new net: J34.4 (C_B), R65.2, U8.16 (B7)
- new net: J33.2 (C_A), R67.2, U8.17 (B6)
- new net: J33.4 (C_B), R69.2, U8.18 (B5)
- new net: J32.2 (C_A), R71.2, U8.19 (B4)
- new net: J32.4 (C_B), R73.2, U8.20 (B3)
- new net: J31.2 (C_A), R75.2, U8.21 (B2)
- new net: J31.4 (C_B), R77.2, U8.22 (B1)
- new net: C11.1, R79.2, U8.23 (VrefB), U8.24 (EN)
- new net: D_TX1.2 (A), R80.2
- new net: D_RX1.2 (A), R81.2
- new net 10a: H1.22 (Pin_22), U3.12 (A10)
- new net 10b: H1.21 (Pin_21), U3.11 (A9)
- new net 11a: H1.24 (Pin_24), U4.4 (A2)
- new net 11b: H1.23 (Pin_23), U4.3 (A1)
- new net 12a: H1.26 (Pin_26), U4.6 (A4)
- new net 12b: H1.25 (Pin_25), U4.5 (A3)
- new net 13a: H1.28 (Pin_28), U4.8 (A6)
- new net 13b: H1.27 (Pin_27), U4.7 (A5)
- new net 14a: H1.32 (Pin_32), U4.10 (A8)
- new net 14b: H1.31 (Pin_31), U4.9 (A7)
- new net 15a: H1.34 (Pin_34), U4.12 (A10)
- new net 15b: H1.33 (Pin_33), U4.11 (A9)
- new net 16a: H1.40 (Pin_40), U5.4 (A2)
- new net 16b: H1.39 (Pin_39), U5.3 (A1)
- new net 17a: H1.38 (Pin_38), U5.6 (A4)
- new net 17b: H1.37 (Pin_37), U5.5 (A3)
- new net 18a: H1.36 (Pin_36), U5.8 (A6)
- new net 18b: H1.35 (Pin_35), U5.7 (A5)
- new net 19a: H2.4 (Pin_4), U5.10 (A8)
- new net 19b: H2.3 (Pin_3), U5.9 (A7)
- new net 1a: H1.2 (Pin_2), U2.4 (A2)
- new net 1b: H1.1 (Pin_1), U2.3 (A1)
- new net 20a: H2.2 (Pin_2), U5.12 (A10)
- new net 20b: H2.1 (Pin_1), U5.11 (A9)
- new net 21a: H2.6 (Pin_6), U6.4 (A2)
- new net 21b: H2.5 (Pin_5), U6.3 (A1)
- new net 22a: H2.8 (Pin_8), U6.6 (A4)
- new net 22b: H2.7 (Pin_7), U6.5 (A3)
- new net 23a: H2.10 (Pin_10), U6.8 (A6)
- new net 23b: H2.9 (Pin_9), U6.7 (A5)
- new net 24a: H2.14 (Pin_14), U6.10 (A8)
- new net 24b: H2.13 (Pin_13), U6.9 (A7)
- new net 25a: H2.16 (Pin_16), U6.12 (A10)
- new net 25b: H2.15 (Pin_15), U6.11 (A9)
- new net 26a: H2.18 (Pin_18), U7.4 (A2)
- new net 26b: H2.17 (Pin_17), U7.3 (A1)
- new net 27a: H2.20 (Pin_20), U7.6 (A4)
- new net 27b: H2.19 (Pin_19), U7.5 (A3)
- new net 28a: H2.22 (Pin_22), U7.8 (A6)
- new net 28b: H2.21 (Pin_21), U7.7 (A5)
- new net 29a: H2.24 (Pin_24), U7.10 (A8)
- new net 29b: H2.23 (Pin_23), U7.9 (A7)
- new net 2a: H1.4 (Pin_4), U2.6 (A4)
- new net 2b: H1.3 (Pin_3), U2.5 (A3)
- new net 30a: H2.26 (Pin_26), U7.12 (A10)
- new net 30b: H2.25 (Pin_25), U7.11 (A9)
- new net 31a: H2.32 (Pin_32), U8.4 (A2)
- new net 31b: H2.28 (Pin_28), U8.3 (A1)
- new net 32a: H2.34 (Pin_34), U8.6 (A4)
- new net 32b: H2.33 (Pin_33), U8.5 (A3)
- new net 33a: H2.36 (Pin_36), U8.8 (A6)
- new net 33b: H2.35 (Pin_35), U8.7 (A5)
- new net 34a: H2.38 (Pin_38), U8.10 (A8)
- new net 34b: H2.37 (Pin_37), U8.9 (A7)
- new net 35a: H2.40 (Pin_40), U8.12 (A10)
- new net 35b: H2.39 (Pin_39), U8.11 (A9)
- new net 3V3: C14.2, C15.2, C16.2, C17.2, C18.2, C19.2, C20.1, H1.29 (Pin_29), H2.29 (Pin_29), J37.7 (Pin_7), U2.2 (VrefA), U3.2 (VrefA), U4.2 (VrefA), U5.2 (VrefA), U6.2 (VrefA), U7.2 (VrefA), U8.2 (VrefA)
- new net 3a: H1.6 (Pin_6), U2.8 (A6)
- new net 3b: H1.5 (Pin_5), U2.7 (A5)
- new net 4a: H1.8 (Pin_8), U2.10 (A8)
- new net 4b: H1.7 (Pin_7), U2.9 (A7)
- new net 5V: C2.1, C21.1, C22.1, C23.1, C24.1, C25.1, C26.1, C27.2, C28.2, C29.2, C3.1, C30.2, C31.2, C4.1, H1.11 (Pin_11), H2.11 (Pin_11), J1.3 (5V), J10.3 (5V), J11.3 (5V), J12.3 (5V), J13.3 (5V), J14.3 (5V), J15.3 (5V), J16.3 (5V), J17.3 (5V), J18.3 (5V), J19.3 (5V), J2.3 (5V), J20.3 (5V), J21.3 (5V), J22.3 (5V), J23.3 (5V), J24.3 (5V), J25.3 (5V), J26.3 (5V), J27.3 (5V), J28.3 (5V), J29.3 (5V), J3.3 (5V), J30.3 (5V), J31.3 (5V), J32.3 (5V), J33.3 (5V), J34.3 (5V), J35.3 (5V), J37.5 (Pin_5), J4.3 (5V), J5.3 (5V), J6.3 (5V), J7.3 (5V), J8.3 (5V), J9.3 (5V), L1.3, R10.1, R11.1, R12.1, R13.1, R14.1, R15.1, R16.1, R17.1, R18.1, R19.1, R20.1, R21.1, R22.1, R23.1, R24.1, R25.1, R26.1, R27.1, R28.1, R29.1, R3.1, R30.1, R31.1, R32.1, R33.1, R34.1, R35.1, R36.1, R37.1, R38.1, R39.1, R4.1, R40.1, R41.1, R42.1, R43.1, R44.1, R45.1, R46.1, R47.1, R48.1, R49.1, R5.1, R50.1, R51.1, R52.1, R53.1, R54.1, R55.1, R56.1, R57.1, R58.1, R59.1, R6.1, R60.1, R61.1, R62.1, R63.1, R64.1, R65.1, R66.1, R67.1, R68.1, R69.1, R7.1, R70.1, R71.1, R72.1, R73.1, R74.1, R75.1, R76.1, R77.1, R78.1, R79.1, R8.1, R80.1, R81.1, R9.1, U1.20 (VCC)
- new net 5a: H1.10 (Pin_10), U2.12 (A10)
- new net 5b: H1.9 (Pin_9), U2.11 (A9)
- new net 6a: H1.14 (Pin_14), U3.4 (A2)
- new net 6b: H1.13 (Pin_13), U3.3 (A1)
- new net 7a: H1.16 (Pin_16), U3.6 (A4)
- new net 7b: H1.15 (Pin_15), U3.5 (A3)
- new net 8a: H1.18 (Pin_18), U3.8 (A6)
- new net 8b: H1.17 (Pin_17), U3.7 (A5)
- new net 9a: H1.20 (Pin_20), U3.10 (A8)
- new net 9b: H1.19 (Pin_19), U3.9 (A7)
- new net GND: C1.2, C10.2, C11.2, C12.2, C13.2, C14.1, C15.1, C16.1, C17.1, C18.1, C19.1, C2.2, C20.2, C21.2, C22.2, C23.2, C24.2, C25.2, C26.2, C27.1, C28.1, C29.1, C3.2, C30.1, C31.1, C4.2, C5.2, C6.2, C7.2, C8.2, C9.2, H1.12 (Pin_12), H1.30 (Pin_30), H2.12 (Pin_12), H2.30 (Pin_30), J0.5 (GND), J0.6 (Shield), J1.1 (GND), J10.1 (GND), J11.1 (GND), J12.1 (GND), J13.1 (GND), J14.1 (GND), J15.1 (GND), J16.1 (GND), J17.1 (GND), J18.1 (GND), J19.1 (GND), J2.1 (GND), J20.1 (GND), J21.1 (GND), J22.1 (GND), J23.1 (GND), J24.1 (GND), J25.1 (GND), J26.1 (GND), J27.1 (GND), J28.1 (GND), J29.1 (GND), J3.1 (GND), J30.1 (GND), J31.1 (GND), J32.1 (GND), J33.1 (GND), J34.1 (GND), J35.1 (GND), J37.8 (Pin_8), J4.1 (GND), J5.1 (GND), J6.1 (GND), J7.1 (GND), J8.1 (GND), J9.1 (GND), L1.2, R2.2, U1.18 (GND), U1.21 (GND), U1.25 (AGND), U1.26 (TEST), U1.7 (GND), U2.1 (GND), U3.1 (GND), U4.1 (GND), U5.1 (GND), U6.1 (GND), U7.1 (GND), U8.1 (GND)
- new net RX: H2.27 (Pin_27), U1.5 (RXD)
- new net TX: H2.31 (Pin_31), U1.1 (TXD)
Other:
- note added: "External oscillator not reqired\nper datasheet when 5V powered.\nFootprint added anyway just in case."
- note added: "TODO:\nresistor values\nmove choke?\nsilkscreen etc\nBNX016-01"
